Commit message: ros2_control CLI

File: src/arduinobot_description/urdf/arduinobot_ros2_control.xacro (robot description, xacro)
@@ -41,9 +41,4 @@
             <state_interface name="position"/>
         </joint>
-        # replicating the joint 4
-        <joint name="joint_5">
-            <param name="mimic">joint_4</param>
-            <param name="multiplier"> -1 </param> # this will help in moving it in the oppsite direction of the joint 4
-        </joint>
     </ros2_control>
 </robot>
